Commit message: Added Nav2 navigation + Slam (not working fully

File: prius_description/urdf/prius.urdf (robot description, URDF)
Before this commit: robot prius, 11 links, 10 joints
Links:
- removed link $(arg namespace)base_link
- removed link $(arg namespace)center_laser_link
- removed link $(arg namespace)chassis
- removed link $(arg namespace)fl_axle
- removed link $(arg namespace)fr_axle
- removed link $(arg namespace)front_left_wheel
- removed link $(arg namespace)front_right_wheel
- removed link $(arg namespace)imu_link
- removed link $(arg namespace)rear_left_wheel
- removed link $(arg namespace)rear_right_wheel
- removed link $(arg namespace)steering_wheel
- added link base_link, mass 1
- added link center_laser_link, mass 0.0
- added link chassis, mass 1356.0; collision box size=1.168381 1.654253 0.272347; collision box size=1.267845 1.116344 0.244286
- added link fl_axle, mass 1
- added link fr_axle, mass 1
- added link front_left_wheel, mass 11; collision sphere radius=0.31265; visual mesh filename=package://prius_description/meshes/wheel.obj scale=0.01 0.01 0.01
- added link front_right_wheel, mass 11; collision sphere radius=0.31265; visual mesh filename=package://prius_description/meshes/wheel.obj scale=0.01 0.01 0.01
- added link imu_link
- added link rear_left_wheel, mass 11; collision sphere radius=0.31265; visual mesh filename=package://prius_description/meshes/wheel.obj scale=0.01 0.01 0.01
- added link rear_right_wheel, mass 11; collision sphere radius=0.31265; visual mesh filename=package://prius_description/meshes/wheel.obj scale=0.01 0.01 0.01
- added link steering_wheel, mass 1.0; visual mesh filename=package://prius_description/meshes/steering_wheel.obj scale=0.01 0.01 0.01
Joints:
- joint base_link_connection: child $(arg namespace)chassis -> chassis; parent $(arg namespace)base_link -> base_link
- joint center_laser_joint: child $(arg namespace)center_laser_link -> center_laser_link; parent $(arg namespace)chassis -> chassis
- joint front_left_steer_joint: child $(arg namespace)fl_axle -> fl_axle; parent $(arg namespace)chassis -> chassis
- joint front_left_wheel_joint: child $(arg namespace)front_left_wheel -> front_left_wheel; parent $(arg namespace)fl_axle -> fl_axle
- joint front_right_steer_joint: child $(arg namespace)fr_axle -> fr_axle; parent $(arg namespace)chassis -> chassis
- joint front_right_wheel_joint: child $(arg namespace)front_right_wheel -> front_right_wheel; parent $(arg namespace)fr_axle -> fr_axle
- joint imu_joint: child $(arg namespace)imu_link -> imu_link; parent $(arg namespace)chassis -> chassis
- joint rear_left_wheel_joint: child $(arg namespace)rear_left_wheel -> rear_left_wheel; parent $(arg namespace)chassis -> chassis
- joint rear_right_wheel_joint: child $(arg namespace)rear_right_wheel -> rear_right_wheel; parent $(arg namespace)chassis -> chassis
- joint steering_joint: child $(arg namespace)steering_wheel -> steering_wheel; parent $(arg namespace)chassis -> chassis
